File: afe.kicad_sch (KiCad schematic)
At the start: 163 parts, among them J1 Conn_01x18, Q1 Q_NMOS_GDS, Q10 Q_NMOS_GDS, Q11 Q_NMOS_GDS, Q12 Q_NMOS_GDS, Q13 Q_NMOS_GDS, Q14 Q_NMOS_GDS, Q15 Q_NMOS_GDS, Q16 Q_NMOS_GDS, Q17 Q_NMOS_GDS, Q18 Q_NMOS_GDS, Q19 Q_NMOS_GDS, Q2 Q_NMOS_GDS, Q20 Q_NMOS_GDS, Q21 Q_NMOS_GDS, Q22 Q_NMOS_GDS, Q23 Q_NMOS_GDS, Q24 Q_NMOS_GDS, Q25 Q_NMOS_GDS, Q26 Q_NMOS_GDS, Q29 Q_NMOS_GDS, Q3 Q_PMOS_GDS, Q30 Q_NMOS_GDS, Q31 Q_NMOS_GDS, Q32 Q_NMOS_GDS, Q33 Q_NMOS_GDS, Q34 Q_NMOS_GDS, Q35 Q_NMOS_GDS, Q36 Q_NMOS_GDS, Q37 Q_NMOS_GDS, Q38 Q_NMOS_GDS, Q4 Q_NPN_BEC, U1 PB7170

Commit message: PCB连接大部分走线，微调原理图
Parts:
- R56: footprint Resistor_SMD:R_0402_1005Metric -> Resistor_SMD:R_0603_1608Metric
Changed lines of the file:
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@@
 			)
 		)
-		(property "Footprint" "Resistor_SMD:R_0402_1005Metric"
+		(property "Footprint" "Resistor_SMD:R_0603_1608Metric"
 			(at 83.82 107.188 90)
 			(effects
