File: bmsboard_17s.kicad_pcb (KiCad board)
At the start: 2 copper layers, 100 x 90 mm, 274 parts, among them J2 Conn_01x08, J3 Conn_01x02, J4 Conn_01x04, J5 Conn_01x02, J6 Conn_01x02, Q1 Q_NMOS_GDS, Q10 Q_NMOS_GDS, Q11 Q_NMOS_GDS, Q12 Q_NMOS_GDS, Q13 Q_NMOS_GDS, Q14 Q_NMOS_GDS, Q15 Q_NMOS_GDS, Q16 Q_NMOS_GDS, Q17 Q_NMOS_GDS, Q18 Q_NMOS_GDS, Q19 Q_NMOS_GDS, Q2 Q_NMOS_GDS, Q20 Q_NMOS_GDS, Q21 Q_NMOS_GDS, Q22 Q_NMOS_GDS, Q23 Q_NMOS_GDS, Q24 Q_NMOS_GDS, Q25 Q_NMOS_GDS, Q26 Q_NMOS_GDS, Q27 PMOS, Q28 PMOS, Q29 Q_NMOS_GDS, Q3 Q_PMOS_GDS, Q30 Q_NMOS_GDS, Q31 Q_NMOS_GDS, Q32 Q_NMOS_GDS, Q33 Q_NMOS_GDS, Q34 Q_NMOS_GDS, Q35 Q_NMOS_GDS, Q36 Q_NMOS_GDS, Q37 Q_NMOS_GDS, Q38 Q_NMOS_GDS, Q4 Q_NPN_BEC, Q5 Q_NPN_BEC, Q6 Q_NPN_BEC, Q7 Q_NPN_BEC, Q8 Q_NPN_BEC, Q9 Q_NPN_BEC, U1 PB7170, U10 TJA1042T-3, U11 MAX485E, U12 PY32F003F1xUx, U13 YX59012, U14 SGM2033-3.3, U2 CH32V103C8T6, U3 XTSD01G, U4 74HC138, U5 BMP280, U7 Si7020-A20, U8 QMA6100P, U9 ADS1243, Y1 16MHz, Y2 32.768kHz

Commit message: PCB连接大部分走线，微调原理图
Parts:
- R56: footprint Resistor_SMD:R_0402_1005Metric -> Resistor_SMD:R_0603_1608Metric
- moved R83 13.1 mm to (102.8, 112.0), turned to 90 degrees
- moved R80 9.65 mm to (102.8, 115.4), turned to 90 degrees
- moved C53 3.77 mm to (97.1, 94.7), turned to -90 degrees
- moved R61 1.14 mm to (98.7, 63.7), turned to 0 degrees
- moved R79 0.92 mm to (113.0, 102.7), turned to -90 degrees
- moved R78 0.85 mm to (113.0, 105.2), turned to -90 degrees
- moved R56 0.65 mm to (74.5, 56.0)
- moved R81 0.59 mm to (113.0, 100.2), turned to -90 degrees
- turned R76 to -90 degrees
- turned U7 to 180 degrees
Connections:
- C49 pad 1: Net-(D42-K) -> +5V
- C50 pad 1: Net-(D42-K) -> +5V
- D42 pad 1: Net-(D42-K) -> +5V
- L3 pad 2: Net-(D42-K) -> +5V
- R100 pad 2: Net-(D42-K) -> +5V
- U14 pad 1: Net-(D42-K) -> +5V
- U14 pad 3: Net-(D42-K) -> +5V
- U2 pad 37: /CS_AFE -> /CS_BLE
- U2 pad 38: /CS_BLE -> /CS_AFE
Routing:
- net +3.3V: track 16.1 -> 205.4 mm, vias 0 -> 4
- net GND: track 108.6 -> 221.8 mm, vias 0 -> 11
- net +5V: track 3.67 -> 62.4 mm, vias 0 -> 4
- net /MISO: track 2.68 -> 53.6 mm, vias 0 -> 2
- net /MOSI: track 0.76 -> 48.9 mm, vias 0 -> 4
- net /SCLK: track 0.83 -> 45.5 mm, vias 0 -> 2
- net /MCU Module/CANRX: track 0.00 -> 35.9 mm, vias 0 -> 1
- net /CS_AFE: track 2.70 -> 36.7 mm
- net /MCU Module/CANTX: track 0.00 -> 30.0 mm, vias 0 -> 1
- net /Sensors Module/SCL: track 0.00 -> 28.4 mm, vias 0 -> 3
- net /Sensors Module/SDA: track 0.00 -> 26.5 mm, vias 0 -> 2
- net Net-(Q28-D): track 0.00 -> 26.0 mm
- net BAT+: track 62.3 -> 38.5 mm
- net Net-(D42-K): track 21.7 -> 0.00 mm, vias 4 -> 0
- net /MCU Module/CANSTB: track 0.00 -> 21.3 mm, vias 0 -> 1
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- added copper zone on F.Cu, net +3.3V
- added copper zone on B.Cu, net GND
- added copper zone on F.Cu, net GND
