File: mcu.kicad_sch (KiCad schematic)
At the start: 69 parts, among them J5 Conn_01x02, J6 Conn_01x02, Q5 Q_NPN_BEC, Q6 Q_NPN_BEC, Q7 Q_NPN_BEC, Q8 Q_NPN_BEC, Q9 Q_NPN_BEC, U10 TJA1042T-3, U11 MAX485E, U2 CH32V103C8T6, U3 XTSD01G, Y1 16MHz, Y2 32.768kHz

Commit message: PCB连接大部分走线，微调原理图
Connections:
- net CS_AFE: now also U2.38 (PA15); no longer U2.37 (PA14)
- net CS_BLE: now also U2.37 (PA14); no longer U2.38 (PA15)
Changed lines of the file:
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@@
 	(hierarchical_label "CS_BLE"
 		(shape output)
-		(at 100.33 119.38 0)
+		(at 100.33 116.84 0)
 		(effects
 			(font
@@
 	(hierarchical_label "CS_AFE"
 		(shape output)
-		(at 100.33 116.84 0)
+		(at 100.33 119.38 0)
 		(effects
 			(font
